File: crossbar/crossbar.kicad_sch (KiCad schematic)
At the start: 22 parts, among them J1 Conn_01x16_Pin, J10 Conn_01x16_Pin, J11 Conn_01x16_Pin, J12 Conn_01x16_Pin, J13 Conn_01x16_Pin, J14 Conn_01x16_Pin, J15 Conn_01x16_Pin, J16 Conn_01x16_Pin, J17 Conn_01x16_Pin, J18 Conn_01x16_Pin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

Commit message: crossbar & terminals
Parts:
- J1: LCSC# (none) -> C2894958
- J10, J11, J12, J13, J14, J15, J16, J17, J18, J3, J4, J5, J6, J7, J8, J9: LCSC# (none) -> C2894939
- J19, J20: LCSC# (none) -> C2894946
- J2: LCSC# (none) -> C2897398
- J21, J22: LCSC# (none) -> C2897386
Changed lines of the file:
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@@
+      (effects (font (size 1.27 1.27)) hide)
+    )
+    (property "LCSC#" "C2894946" (at 99.06 31.75 0)
       (effects (font (size 1.27 1.27)) hide)
     )
@@
       (effects (font (size 1.27 1.27)) hide)
     )
+    (property "LCSC#" "C2894939" (at 109.22 62.23 0)
+      (effects (font (size 1.27 1.27)) hide)
+    )
     (pin "1")
     (pin "10")
@@
       (effects (font (size 1.27 1.27)) hide)
     )
+    (property "LCSC#" "C2894939" (at 109.22 173.99 0)
+      (effects (font (size 1.27 1.27)) hide)
+    )
     (pin "1")
     (pin "10")
@@
     )
     (property "Datasheet" "~" (at 109.22 102.87 0)
+      (effects (font (size 1.27 1.27)) hide)
+    )
+    (property "LCSC#" "C2894939" (at 109.22 102.87 0)
       (effects (font (size 1.27 1.27)) hide)
     )
@@
       (effects (font (size 1.27 1.27)) hide)
     )
+    (property "LCSC#" "C2894958" (at 55.88 125.73 0)
+      (effects (font (size 1.27 1.27)) hide)
+    )
     (pin "1")
     (pin "10")
@@
       (effects (font (size 1.27 1.27)) hide)
     )
+    (property "LCSC#" "C2894939" (at 109.22 52.07 0)
+      (effects (font (size 1.27 1.27)) hide)
+    )
     (pin "1")
     (pin "10")
@@
       (effects (font (size 1.27 1.27)) hide)
     )
+    (property "LCSC#" "C2894939" (at 109.22 184.15 0)
+      (effects (font (size 1.27 1.27)) hide)
+    )
     (pin "1")
     (pin "10")
@@
       (effects (font (size 1.27 1.27)) hide)
     )
+    (property "LCSC#" "C2894939" (at 109.22 163.83 0)
+      (effects (font (size 1.27 1.27)) hide)
+    )
     (pin "1")
     (pin "10")
@@
     )
     (property "Datasheet" "~" (at 109.22 123.19 0)
+      (effects (font (size 1.27 1.27)) hide)
+    )
+    (property "LCSC#" "C2894939" (at 109.22 123.19 0)
       (effects (font (size 1.27 1.27)) hide)
     )
@@
       (effects (font (size 1.27 1.27)) hide)
     )
+    (property "LCSC#" "C2897386" (at 99.06 217.17 0)
+      (effects (font (size 1.27 1.27)) hide)
+    )
     (pin "1")
     (pin "2")
@@
       (effects (font (size 1.27 1.27)) hide)
     )
+    (property "LCSC#" "C2894939" (at 109.22 143.51 0)
+      (effects (font (size 1.27 1.27)) hide)
+    )
     (pin "1")
     (pin "10")
@@
       (effects (font (size 1.27 1.27)) hide)
     )
+    (property "LCSC#" "C2894939" (at 109.22 72.39 0)
+      (effects (font (size 1.27 1.27)) hide)
+    )
     (pin "1")
     (pin "10")
@@
     )
     (property "Datasheet" "~" (at 109.22 113.03 0)
+      (effects (font (size 1.27 1.27)) hide)
+    )
+    (property "LCSC#" "C2894939" (at 109.22 113.03 0)
       (effects (font (size 1.27 1.27)) hide)
     )
@@
       (effects (font (size 1.27 1.27)) hide)
     )
+    (property "LCSC#" "C2897386" (at 119.38 217.17 0)
+      (effects (font (size 1.27 1.27)) hide)
+    )
     (pin "1")
     (pin "2")
@@
       (effects (font (size 1.27 1.27)) hide)
     )
+    (property "LCSC#" "C2894939" (at 109.22 153.67 0)
+      (effects (font (size 1.27 1.27)) hide)
+    )
     (pin "1")
     (pin "10")
@@
       (effects (font (size 1.27 1.27)) hide)
     )
+    (property "LCSC#" "C2894939" (at 109.22 82.55 0)
+      (effects (font (size 1.27 1.27)) hide)
+    )
     (pin "1")
     (pin "10")
@@
     )
     (property "Datasheet" "~" (at 109.22 133.35 0)
+      (effects (font (size 1.27 1.27)) hide)
+    )
+    (property "LCSC#" "C2894939" (at 109.22 133.35 0)
       (effects (font (size 1.27 1.27)) hide)
     )
@@
       (effects (font (size 1.27 1.27)) hide)
     )
+    (property "LCSC#" "C2897398" (at 165.1 125.73 0)
+      (effects (font (size 1.27 1.27)) hide)
+    )
     (pin "1")
     (pin "10")
@@
       (effects (font (size 1.27 1.27)) hide)
     )
+    (property "LCSC#" "C2894939" (at 109.22 194.31 0)
+      (effects (font (size 1.27 1.27)) hide)
+    )
     (pin "1")
     (pin "10")
@@
       (effects (font (size 1.27 1.27)) hide)
     )
+    (property "LCSC#" "C2894939" (at 109.22 92.71 0)
+      (effects (font (size 1.27 1.27)) hide)
+    )
     (pin "1")
     (pin "10")
@@
     )
     (property "Datasheet" "~" (at 109.22 204.47 0)
+      (effects (font (size 1.27 1.27)) hide)
+    )
+    (property "LCSC#" "C2894939" (at 109.22 204.47 0)
       (effects (font (size 1.27 1.27)) hide)
     )
@@
       (effects (font (size 1.27 1.27)) hide)
     )
+    (property "LCSC#" "C2894946" (at 119.38 31.75 0)
+      (effects (font (size 1.27 1.27)) hide)
+    )
